File: Docs/KiCad/mains_mon_test_ckt_1.kicad_sch (KiCad schematic)
At the start: 18 parts, among them Q1 NMOS, T1 10:1, U1 HLW8032

Commit message: Update schematic
Parts:
- removed F1: Fuse, symbol Device:Fuse
- removed LOAD: 6.5R 10W, symbol Device:R
- removed Q1: NMOS, symbol Simulation_SPICE:NMOS
- removed R3: 300m, symbol Device:R
- removed T1: 10:1, symbol Device:Transformer_1P_1S
- added J1: Barrel_Jack, symbol Connector:Barrel_Jack
- R1: value 300m -> 5K1
- R2: value 300m -> 10K
- R8: value 10k -> 100m
- R9: value 10k -> 20
Connections:
- net +5V: no longer R8.1
- net 12VAC: now also R5.1, R6.2, R8.1, J1.1; no longer R1.1, R2.1, R4.1, R6.1
- net GND: now also R2.1, R9.2, U1.5 (GND), J1.2; no longer R1.2, R2.2, R5.1
- net GND1: no longer U1.5 (GND)
- net VP: now also R6.1; no longer R6.2
- net +3V3: no longer names the net of R9.1
- net +3V3: now also R4.1, R8.2; no longer A1.2 (3V3)
- net HLW_TX renamed DATA_5V
- net DATA_5V: now also R1.1; no longer R8.2
- net IO16 renamed DATA_3V3
- net DATA_3V3: now also R1.2, R2.2; no longer R9.2
- no-connect marks 25 -> 26
Other:
- note added: "12VAC at 1.5A"
- note added: "Controller"
- note added: "HLW8032"
- note added: "High percision current shunt"
- note added: "Load"
- note added: "Power"
- note added: "Power Monitoring"
- note added: "Rated for 10W"
- note added: "esp32 connected to PC for power and logging"
- note removed: "5v-3v3 Level Shifter"
- note removed: "AC-AC 12VAC 1.5A Wall Adapter"
- note removed: "Current Shunt"
- note removed: "Differential Current Input"
- note removed: "ESP32 Huzzah"
- note removed: "HLW8032 Energy Meter"
- note removed: "Test Load"
- note removed: "Voltage Divider"
- note removed: "https://www.jameco.com/Jameco/Products/ProdDS/167151.pdf"
- moved on the sheet: A1, C1, C2, C3, R4, R5, R6, R7, U1
